Commit message: accurate description

File: src/picar_description/urdf/picar.urdf.xacro (robot description, xacro)
@@ -10,5 +10,5 @@
     <parent link="base_link"/>
     <child link="rear_left_wheel"/>
-    <origin xyz="0 0.1 0" rpy="0 0 0"/>
+    <origin xyz="0 0.053 -0.015" rpy="0 0 0"/>
     <axis xyz="0 1 0"/>
   </joint>
@@ -16,13 +16,21 @@
     <parent link="base_link"/>
     <child link="rear_right_wheel"/>
-    <origin xyz="0 -0.1 0" rpy="0 0 0"/>
+    <origin xyz="0 -0.053 -0.015" rpy="0 0 0"/>
     <axis xyz="0 1 0"/>
   </joint>
   <!-- steering axle -->
-  <link name="front_axle_link"/>
-  <joint name="steering_joint" type="revolute">
+  <link name="left_axle_link"/>
+  <link name="right_axle_link"/>
+  <joint name="left_steering_joint" type="revolute">
     <parent link="base_link"/>
-    <child link="front_axle_link"/>
-    <origin xyz="0.15 0 0" rpy="0 0 0"/>
+    <child link="left_axle_link"/>
+    <origin xyz="0.14 0.048 -0.015" rpy="0 0 0"/>
+    <axis xyz="0 0 1"/>
+    <limit lower="-0.6" upper="0.6" effort="1" velocity="1"/>
+  </joint>
+  <joint name="right_steering_joint" type="revolute">
+    <parent link="base_link"/>
+    <child link="right_axle_link"/>
+    <origin xyz="0.14 -0.048 -0.015" rpy="0 0 0"/>
     <axis xyz="0 0 1"/>
     <limit lower="-0.6" upper="0.6" effort="1" velocity="1"/>
@@ -32,13 +40,13 @@
   <link name="front_right_wheel"/>
   <joint name="front_left_wheel_joint" type="continuous">
-    <parent link="front_axle_link"/>
+    <parent link="left_axle_link"/>
     <child link="front_left_wheel"/>
-    <origin xyz="0 0.1 0" rpy="0 0 0"/>
+    <origin xyz="0 0.01 0" rpy="0 0 0"/>
     <axis xyz="0 1 0"/>
   </joint>
   <joint name="front_right_wheel_joint" type="continuous">
-    <parent link="front_axle_link"/>
+    <parent link="right_axle_link"/>
     <child link="front_right_wheel"/>
-    <origin xyz="0 -0.1 0" rpy="0 0 0"/>
+    <origin xyz="0 -0.01 0" rpy="0 0 0"/>
     <axis xyz="0 1 0"/>
   </joint>

Commit message: visual in description

File: src/picar_description/urdf/picar.urdf.xacro (robot description, xacro)
@@ -3,8 +3,29 @@
   <!-- test tf tree -->
   <!-- base link -->
-  <link name="base_link"/>
+  <link name="base_link">
+    <visual>
+      <origin xyz="0.064 0 0" />
+      <geometry>
+        <box size="0.21 0.078 0.002"/>
+      </geometry>
+    </visual>
+  </link>
   <!-- rear wheels -->
-  <link name="rear_left_wheel"/>
-  <link name="rear_right_wheel"/>
+  <link name="rear_left_wheel">
+    <visual>
+      <geometry>
+        <cylinder radius="0.033" length="0.025"/>
+      </geometry>
+      <origin rpy="1.5708 0 0"/>
+    </visual>
+  </link>
+  <link name="rear_right_wheel">
+    <visual>
+      <geometry>
+        <cylinder radius="0.033" length="0.025"/>
+      </geometry>
+      <origin rpy="1.5708 0 0"/>
+    </visual>
+  </link>
   <joint name="rear_left_wheel_joint" type="continuous">
     <parent link="base_link"/>
@@ -37,6 +58,20 @@
   </joint>
   <!-- front wheels attached to steering axle -->
-  <link name="front_left_wheel"/>
-  <link name="front_right_wheel"/>
+  <link name="front_left_wheel">
+    <visual>
+      <geometry>
+        <cylinder radius="0.033" length="0.025"/>
+      </geometry>
+      <origin rpy="1.5708 0 0"/>
+    </visual>
+  </link>
+  <link name="front_right_wheel">
+    <visual>
+      <geometry>
+        <cylinder radius="0.033" length="0.025"/>
+      </geometry>
+      <origin rpy="1.5708 0 0"/>
+    </visual>
+  </link>
   <joint name="front_left_wheel_joint" type="continuous">
     <parent link="left_axle_link"/>

Commit message: update tf tree w/ sensors

File: src/picar_description/urdf/picar.urdf.xacro (robot description, xacro)
@@ -5,7 +5,7 @@
   <link name="base_link">
     <visual>
-      <origin xyz="0.064 0 0" />
+      <origin xyz="0.045 0 0" />
       <geometry>
-        <box size="0.21 0.078 0.002"/>
+        <box size="0.18 0.08 0.002"/>
       </geometry>
     </visual>
@@ -31,5 +31,5 @@
     <parent link="base_link"/>
     <child link="rear_left_wheel"/>
-    <origin xyz="0 0.053 -0.015" rpy="0 0 0"/>
+    <origin xyz="0 0.06 -0.015" rpy="0 0 0"/>
     <axis xyz="0 1 0"/>
   </joint>
@@ -37,5 +37,5 @@
     <parent link="base_link"/>
     <child link="rear_right_wheel"/>
-    <origin xyz="0 -0.053 -0.015" rpy="0 0 0"/>
+    <origin xyz="0 -0.06 -0.015" rpy="0 0 0"/>
     <axis xyz="0 1 0"/>
   </joint>
@@ -46,5 +46,5 @@
     <parent link="base_link"/>
     <child link="left_axle_link"/>
-    <origin xyz="0.14 0.048 -0.015" rpy="0 0 0"/>
+    <origin xyz="0.095 0.043 -0.015" rpy="0 0 0"/>
     <axis xyz="0 0 1"/>
     <limit lower="-0.6" upper="0.6" effort="1" velocity="1"/>
@@ -53,5 +53,5 @@
     <parent link="base_link"/>
     <child link="right_axle_link"/>
-    <origin xyz="0.14 -0.048 -0.015" rpy="0 0 0"/>
+    <origin xyz="0.095 -0.043 -0.015" rpy="0 0 0"/>
     <axis xyz="0 0 1"/>
     <limit lower="-0.6" upper="0.6" effort="1" velocity="1"/>
@@ -86,3 +86,28 @@
     <axis xyz="0 1 0"/>
   </joint>
+  <!-- sensor positions -->
+  <link name="sonar_sensor">
+   <visual>
+      <geometry>
+        <box size="0.015 0.06 0.02"/>
+      </geometry>
+    </visual>
+  </link>
+  <joint name="sonar_sensor_joint" type="fixed">
+    <parent link="base_link"/>
+    <child link="sonar_sensor"/>
+    <origin xyz="0.14 0 -0.01" rpy="0 0 0"/>
+  </joint>
+  <link name="grayscale_sensor">
+   <visual>
+      <geometry>
+        <box size="0.06 0.02 0.001"/>
+      </geometry>
+    </visual>
+  </link>
+  <joint name="grayscale_sensor_joint" type="fixed">
+    <parent link="base_link"/>
+    <child link="grayscale_sensor"/>
+    <origin xyz="0.15 0 -0.03" rpy="0 3.14159 1.57079"/>
+  </joint>
 </robot>
